File: hardware/esp8266_fan_control_board.sch (KiCad schematic (older format))
At the start: 0 parts

Commit message: update,
Changed lines of the file:
@@
 EESchema Schematic File Version 4
 LIBS:esp8266_fan_control_board-cache
+LIBS:CH340T-tryout-cache
+LIBS:AMS1117-cache
 EELAYER 29 0
 EELAYER END
 $Descr User 8500 5500
 encoding utf-8
-Sheet 1 9
+Sheet 1 10
 Title ""
 Date ""
@@
 $EndSheet
 $Sheet
-S 750  4400 650  350
+S 850  3650 650  600
 U 5CF23C30
 F0 "power" 50
@@
 Wire Wire Line
 	4600 1450 5050 1450
+$Sheet
+S 1800 1550 650  500
+U 5D0F9966
+F0 "motor" 50
+F1 "motor.sch" 50
+F2 "PWM_IN" I R 2450 1700 50
+$EndSheet
 Wire Bus Line
 	3250 950  3250 1600

Commit message: update,
Changed lines of the file:
@@
 EESchema Schematic File Version 4
 LIBS:esp8266_fan_control_board-cache
-LIBS:CH340T-tryout-cache
-LIBS:AMS1117-cache
+LIBS:FAN0-cache
+LIBS:SHT30_tryout-cache
 EELAYER 29 0
 EELAYER END
@@
 F6 "GPIO13" I R 4600 1950 50
 F7 "WS2812_OUT" O R 4600 1450 50
+F8 "FAN_PWM" I L 3750 1650 50
 $EndSheet
 $Sheet
@@
 F0 "motor" 50
 F1 "motor.sch" 50
-F2 "PWM_IN" I R 2450 1700 50
+F2 "FAN0_EN" I R 2450 1800 50
 $EndSheet
+Entry Wire Line
+	3150 1800 3250 1900
+Wire Wire Line
+	2450 1800 3150 1800
+Text Label 3050 1800 2    50   ~ 0
+FAN0
+Entry Wire Line
+	3250 1750 3350 1650
+Wire Wire Line
+	3350 1650 3750 1650
+Text Label 3450 1650 0    50   ~ 0
+FAN0
 Wire Bus Line
-	3250 950  3250 1600
+	3250 950  3250 2100
 $EndSCHEMATC
