File: hardware/rotary_encoder.sch (KiCad schematic (older format))
At the start: 8 parts, among them J4 ROT_ENC_HEADER, SW6 EC11_VERTICAL

Commit message: update,
Other:
- moved on the sheet: C10, C8, C9, R17, R18, R19
Changed lines of the file:
@@
 EESchema Schematic File Version 4
 LIBS:esp8266_fan_control_board-cache
+LIBS:CH340T-tryout-cache
+LIBS:AMS1117-cache
 EELAYER 29 0
 EELAYER END
 $Descr User 8500 5500
 encoding utf-8
-Sheet 6 9
+Sheet 8 10
 Title ""
 Date ""
@@
 L taobao-r:R273,0603 R17
 U 1 1 5CED60AF
-P 3150 2300
-F 0 "R17" V 2900 2300 50  0000 C CNN
-F 1 "R273,0603" V 3000 2300 50  0000 C CNN
-F 2 "Resistor_SMD:R_0603_1608Metric_Pad1.05x0.95mm_HandSolder" H 3150 2300 50  0001 C CNN
-F 3 "~" H 3150 2300 50  0001 C CNN
-	1    3150 2300
+P 2750 2600
+F 0 "R17" V 2500 2600 50  0000 C CNN
+F 1 "R273,0603" V 2600 2600 50  0000 C CNN
+F 2 "Resistor_SMD:R_0603_1608Metric_Pad1.05x0.95mm_HandSolder" H 2750 2600 50  0001 C CNN
+F 3 "~" H 2750 2600 50  0001 C CNN
+	1    2750 2600
 	0    1    1    0
 $EndComp
@@
 L taobao-r:R273,0603 R18
 U 1 1 5CED6622
-P 3150 2800
-F 0 "R18" V 2900 2800 50  0000 C CNN
-F 1 "R273,0603" V 3000 2800 50  0000 C CNN
-F 2 "Resistor_SMD:R_0603_1608Metric_Pad1.05x0.95mm_HandSolder" H 3150 2800 50  0001 C CNN
-F 3 "~" H 3150 2800 50  0001 C CNN
-	1    3150 2800
-	0    1    1    0
+P 3400 3050
+F 0 "R18" H 3500 3100 50  0000 L CNN
+F 1 "R273,0603" H 3500 3050 50  0000 L CNN
+F 2 "Resistor_SMD:R_0603_1608Metric_Pad1.05x0.95mm_HandSolder" H 3400 3050 50  0001 C CNN
+F 3 "~" H 3400 3050 50  0001 C CNN
+	1    3400 3050
+	1    0    0    -1
 $EndComp
 $Comp
 L taobao-r:R273,0603 R19
 U 1 1 5CED67EF
-P 3150 3250
-F 0 "R19" V 2900 3250 50  0000 C CNN
-F 1 "R273,0603" V 3000 3250 50  0000 C CNN
-F 2 "Resistor_SMD:R_0603_1608Metric_Pad1.05x0.95mm_HandSolder" H 3150 3250 50  0001 C CNN
-F 3 "~" H 3150 3250 50  0001 C CNN
-	1    3150 3250
-	0    1    1    0
+P 4400 3000
+F 0 "R19" H 4500 3050 50  0000 L CNN
+F 1 "R273,0603" H 4500 3000 50  0000 L CNN
+F 2 "Resistor_SMD:R_0603_1608Metric_Pad1.05x0.95mm_HandSolder" H 4400 3000 50  0001 C CNN
+F 3 "~" H 4400 3000 50  0001 C CNN
+	1    4400 3000
+	-1   0    0    -1
 $EndComp
 $Comp
 L taobao-c:C104,0603 C10
 U 1 1 5CED6CD1
-P 2800 3450
-F 0 "C10" H 2900 3500 50  0000 L CNN
-F 1 "C104,0603" H 2900 3450 50  0000 L CNN
-F 2 "Capacitor_SMD:C_0603_1608Metric_Pad1.05x0.95mm_HandSolder" H 2800 3450 50  0001 C CNN
-F 3 "~" H 2800 3450 50  0001 C CNN
-	1    2800 3450
-	1    0    0    -1
+P 4400 3450
+F 0 "C10" H 4300 3500 50  0000 R CNN
+F 1 "C104,0603" H 4300 3450 50  0000 R CNN
+F 2 "Capacitor_SMD:C_0603_1608Metric_Pad1.05x0.95mm_HandSolder" H 4400 3450 50  0001 C CNN
+F 3 "~" H 4400 3450 50  0001 C CNN
+	1    4400 3450
+	-1   0    0    -1
 $EndComp
 $Comp
 L taobao-c:C104,0603 C9
 U 1 1 5CED7298
-P 2800 2950
-F 0 "C9" H 2900 3000 50  0000 L CNN
-F 1 "C104,0603" H 2900 2950 50  0000 L CNN
-F 2 "Capacitor_SMD:C_0603_1608Metric_Pad1.05x0.95mm_HandSolder" H 2800 2950 50  0001 C CNN
-F 3 "~" H 2800 2950 50  0001 C CNN
-	1    2800 2950
+P 3400 3400
+F 0 "C9" H 3500 3450 50  0000 L CNN
+F 1 "C104,0603" H 3500 3400 50  0000 L CNN
+F 2 "Capacitor_SMD:C_0603_1608Metric_Pad1.05x0.95mm_HandSolder" H 3400 3400 50  0001 C CNN
+F 3 "~" H 3400 3400 50  0001 C CNN
+	1    3400 3400
 	1    0    0    -1
 $EndComp
@@
 L taobao-c:C104,0603 C8
 U 1 1 5CED75A5
-P 2800 2500
-F 0 "C8" H 2900 2550 50  0000 L CNN
-F 1 "C104,0603" H 2900 2500 50  0000 L CNN
-F 2 "Capacitor_SMD:C_0603_1608Metric_Pad1.05x0.95mm_HandSolder" H 2800 2500 50  0001 C CNN
-F 3 "~" H 2800 2500 50  0001 C CNN
-	1    2800 2500
+P 2400 2800
+F 0 "C8" H 2500 2850 50  0000 L CNN
+F 1 "C104,0603" H 2500 2800 50  0000 L CNN
+F 2 "Capacitor_SMD:C_0603_1608Metric_Pad1.05x0.95mm_HandSolder" H 2400 2800 50  0001 C CNN
+F 3 "~" H 2400 2800 50  0001 C CNN
+	1    2400 2800
 	1    0    0    -1
 $EndComp
 Wire Wire Line
-	3050 2300 2800 2300
-Wire Wire Line
-	2800 2300 2800 2400
-Wire Wire Line
-	3050 2800 2800 2800
-Wire Wire Line
-	2800 2800 2800 2850
-Wire Wire Line
-	3050 3250 2800 3250
-Wire Wire Line
-	2800 3250 2800 3350
+	2650 2600 2400 2600
+Wire Wire Line
+	2400 2600 2400 2700
+Wire Wire Line
+	3400 3150 3400 3250
+Wire Wire Line
+	3400 3250 3400 3300
+Wire Wire Line
+	4400 3100 4400 3250
+Wire Wire Line
+	4400 3250 4400 3350
 $Comp
 L power:GND #PWR0135
 U 1 1 5CED86F3
-P 2800 2650
-F 0 "#PWR0135" H 2800 2400 50  0001 C CNN
-F 1 "GND" H 2850 2450 50  0000 C CNN
-F 2 "" H 2800 2650 50  0001 C CNN
-F 3 "" H 2800 2650 50  0001 C CNN
-	1    2800 2650
+P 2400 2950
+F 0 "#PWR0135" H 2400 2700 50  0001 C CNN
+F 1 "GND" H 2450 2750 50  0000 C CNN
+F 2 "" H 2400 2950 50  0001 C CNN
+F 3 "" H 2400 2950 50  0001 C CNN
+	1    2400 2950
 	1    0    0    -1
 $EndComp
 Wire Wire Line
-	2800 2650 2800 2600
+	2400 2950 2400 2900
 $Comp
 L power:GND #PWR0136
 U 1 1 5CED8B04
-P 2800 3100
-F 0 "#PWR0136" H 2800 2850 50  0001 C CNN
-F 1 "GND" H 2850 2900 50  0000 C CNN
-F 2 "" H 2800 3100 50  0001 C CNN
-F 3 "" H 2800 3100 50  0001 C CNN
-	1    2800 3100
+P 3400 3550
+F 0 "#PWR0136" H 3400 3300 50  0001 C CNN
+F 1 "GND" H 3450 3350 50  0000 C CNN
+F 2 "" H 3400 3550 50  0001 C CNN
+F 3 "" H 3400 3550 50  0001 C CNN
+	1    3400 3550
 	1    0    0    -1
 $EndComp
 Wire Wire Line
-	2800 3100 2800 3050
+	3400 3550 3400 3500
 $Comp
 L power:GND #PWR0137
 U 1 1 5CED8F95
-P 2800 3600
-F 0 "#PWR0137" H 2800 3350 50  0001 C CNN
-F 1 "GND" H 2850 3400 50  0000 C CNN
-F 2 "" H 2800 3600 50  0001 C CNN
-F 3 "" H 2800 3600 50  0001 C CNN
-	1    2800 3600
-	1    0    0    -1
+P 4400 3600
+F 0 "#PWR0137" H 4400 3350 50  0001 C CNN
+F 1 "GND" H 4450 3400 50  0000 C CNN
+F 2 "" H 4400 3600 50  0001 C CNN
+F 3 "" H 4400 3600 50  0001 C CNN
+	1    4400 3600
+	-1   0    0    -1
 $EndComp
 Wire Wire Line
-	2800 3600 2800 3550
+	4400 3600 4400 3550
 $Comp
 L power:GND #PWR0138
 U 1 1 5CED947F
-P 3350 2600
-F 0 "#PWR0138" H 3350 2350 50  0001 C CNN
-F 1 "GND" H 3400 2400 50  0000 C CNN
-F 2 "" H 3350 2600 50  0001 C CNN
-F 3 "" H 3350 2600 50  0001 C CNN
-	1    3350 2600
-	-1   0    0    1
+P 3150 2950
+F 0 "#PWR0138" H 3150 2700 50  0001 C CNN
+F 1 "GND" H 3200 2750 50  0000 C CNN
+F 2 "" H 3150 2950 50  0001 C CNN
+F 3 "" H 3150 2950 50  0001 C CNN
+	1    3150 2950
+	-1   0    0    -1
 $EndComp
 $Comp
 L power:GND #PWR0139
 U 1 1 5CED96CA
-P 4400 2900
-F 0 "#PWR0139" H 4400 2650 50  0001 C CNN
-F 1 "GND" H 4450 2700 50  0000 C CNN
-F 2 "" H 4400 2900 50  0001 C CNN
-F 3 "" H 4400 2900 50  0001 C CNN
-	1    4400 2900
-	1    0    0    -1
+P 4400 2300
+F 0 "#PWR0139" H 4400 2050 50  0001 C CNN
+F 1 "GND" H 4450 2100 50  0000 C CNN
+F 2 "" H 4400 2300 50  0001 C CNN
+F 3 "" H 4400 2300 50  0001 C CNN
+	1    4400 2300
+	1    0    0    1
 $EndComp
 Wire Wire Line
 	4200 2600 4400 2600
 Wire Wire Line
-	4400 2600 4400 2900
-Wire Wire Line
-	3350 2600 3350 2700
-Wire Wire Line
-	3600 2600 3450 2600
-Wire Wire Line
-	3450 2600 3450 2300
-Wire Wire Line
-	3450 2300 3250 2300
-Wire Wire Line
-	3350 2700 3600 2700
-Wire Wire Line
-	3600 2800 3250 2800
-Wire Wire Line
-	4200 2800 4300 2800
-Wire Wire Line
-	4300 2800 4300 3250
-Wire Wire Line
-	4300 3250 3250 3250
-Text Label 2000 2300 0    50   ~ 0
+	4400 2600 4400 2300
+Wire Wire Line
+	4200 2800 4400 2800
+Text Label 1600 2600 0    50   ~ 0
 ROT_ENC_A
-Text Label 2000 2800 0    50   ~ 0
+Text Label 2600 3250 0    50   ~ 0
 ROT_ENC_B
-Text Label 2000 3250 0    50   ~ 0
+Text Label 5200 3250 2    50   ~ 0
 ROT_ENC_SW
 Wire Wire Line
-	2000 2300 2800 2300
-Connection ~ 2800 2300
-Wire Wire Line
-	2000 2800 2800 2800
-Connection ~ 2800 2800
-Wire Wire Line
-	2000 3250 2800 3250
-Connection ~ 2800 3250
+	1600 2600 2400 2600
+Connection ~ 2400 2600
+Wire Wire Line
+	2600 3250 3400 3250
+Connection ~ 3400 3250
+Wire Wire Line
+	5200 3250 4400 3250
+Connection ~ 4400 3250
 $Comp
 L Connector:Conn_01x03_Female J4
@@
 Wire Wire Line
 	1800 2300 1300 2300
+Wire Wire Line
+	4400 2900 4400 2800
+Wire Wire Line
+	3600 2800 3400 2800
+Wire Wire Line
+	3400 2800 3400 2950
+Wire Wire Line
+	3150 2950 3150 2700
+Wire Wire Line
+	3150 2700 3600 2700
+Wire Wire Line
+	2850 2600 3600 2600
 $EndSCHEMATC
