File: hardware/CH340T.sch (KiCad schematic (older format))
At the start: 11 parts

Commit message: update,
Parts:
- gave numbers to parts that had none: 11
Changed lines of the file:
@@
 $EndDescr
 $Comp
-L taobao-components:USB_Micro U?
+L taobao-components:USB_Micro U4
 U 1 1 5D058DA8
 P 2100 2300
-F 0 "U?" H 2100 2765 50  0000 C CNN
+F 0 "U4" H 2100 2765 50  0000 C CNN
 F 1 "USB_Micro" H 2100 2674 50  0000 C CNN
 F 2 "footprint-lib:USB_Micro-B_Molex-105017-0001" H 2100 1800 50  0001 C CNN
@@
 $EndComp
 $Comp
-L taobao-components:CH340T U?
+L taobao-components:CH340T U3
 U 1 1 5D05D663
 P 4900 2150
-F 0 "U?" H 4875 3093 60  0000 C CNN
+F 0 "U3" H 4875 3093 60  0000 C CNN
 F 1 "CH340T" H 4875 2987 60  0000 C CNN
 F 2 "footprint-lib:CH340T_SSOP-20" H 4875 2881 60  0001 C CNN
@@
 $EndComp
 $Comp
-L taobao-osc:O_12M,3225 Y?
+L taobao-osc:O_12M,3225 Y1
 U 1 1 5D05E9C1
 P 3600 2700
-F 0 "Y?" H 3600 2925 50  0000 C CNN
+F 0 "Y1" H 3600 2925 50  0000 C CNN
 F 1 "O_12M,3225" H 3600 2834 50  0000 C CNN
 F 2 "footprint-lib:OSC_3225" H 3600 2700 50  0001 C CNN
@@
 	3400 2700 3500 2700
 $Comp
-L taobao-c:C22pf,0603 C?
+L taobao-c:C22pf,0603 C11
 U 1 1 5D061A62
 P 3400 2900
-F 0 "C?" H 3300 2950 50  0000 R CNN
+F 0 "C11" H 3300 2950 50  0000 R CNN
 F 1 "C22pf,0603" H 3300 2900 50  0000 R CNN
 F 2 "Capacitor_SMD:C_0603_1608Metric_Pad1.05x0.95mm_HandSolder" H 3400 2900 50  0001 C CNN
@@
 $EndComp
 $Comp
-L taobao-c:C22pf,0603 C?
+L taobao-c:C22pf,0603 C12
 U 1 1 5D06326C
 P 3850 2900
-F 0 "C?" H 3942 2946 50  0000 L CNN
+F 0 "C12" H 3942 2946 50  0000 L CNN
 F 1 "C22pf,0603" H 3942 2855 50  0000 L CNN
 F 2 "Capacitor_SMD:C_0603_1608Metric_Pad1.05x0.95mm_HandSolder" H 3850 2900 50  0001 C CNN
@@
 Connection ~ 3400 2700
 $Comp
-L power:GND #PWR?
+L power:GND #PWR0121
 U 1 1 5D0658C0
 P 3650 3200
-F 0 "#PWR?" H 3650 2950 50  0001 C CNN
+F 0 "#PWR0121" H 3650 2950 50  0001 C CNN
 F 1 "GND" H 3655 3027 50  0000 C CNN
 F 2 "" H 3650 3200 50  0001 C CNN
@@
 	3550 3100 3650 3100
 $Comp
-L taobao-c:C103,0603 C?
+L taobao-c:C103,0603 C7
 U 1 1 5D06DB24
 P 3950 1850
-F 0 "C?" H 4042 1896 50  0000 L CNN
+F 0 "C7" H 4042 1896 50  0000 L CNN
 F 1 "C103,0603" H 4042 1805 50  0000 L CNN
 F 2 "Capacitor_SMD:C_0603_1608Metric_Pad1.05x0.95mm_HandSolder" H 3950 1850 50  0001 C CNN
@@
 $EndComp
 $Comp
-L taobao-c:C104,0603 C?
+L taobao-c:C104,0603 C6
 U 1 1 5D06F240
 P 3450 1850
-F 0 "C?" H 3500 2050 50  0000 L CNN
+F 0 "C6" H 3500 2050 50  0000 L CNN
 F 1 "C104,0603" H 3500 1950 50  0000 L CNN
 F 2 "Capacitor_SMD:C_0603_1608Metric_Pad1.05x0.95mm_HandSolder" H 3450 1850 50  0001 C CNN
@@
 $EndComp
 $Comp
-L taobao-c:C225,0603 C?
+L taobao-c:C225,0603 C5
 U 1 1 5D06FAA1
 P 3200 1850
-F 0 "C?" H 3150 2300 50  0000 L CNN
+F 0 "C5" H 3150 2300 50  0000 L CNN
 F 1 "C225,0603" H 3150 2200 50  0000 L CNN
 F 2 "Capacitor_SMD:C_0603_1608Metric_Pad1.05x0.95mm_HandSolder" H 3200 1850 50  0001 C CNN
@@
 Connection ~ 3450 2000
 $Comp
-L power:GND #PWR?
+L power:GND #PWR0122
 U 1 1 5D0758C8
 P 3650 2050
-F 0 "#PWR?" H 3650 1800 50  0001 C CNN
+F 0 "#PWR0122" H 3650 1800 50  0001 C CNN
 F 1 "GND" H 3655 1877 50  0000 C CNN
 F 2 "" H 3650 2050 50  0001 C CNN
@@
 	3950 1700 3950 1750
 $Comp
-L Connector:Conn_01x10_Female J?
+L Connector:Conn_01x10_Female J5
 U 1 1 5D097AD0
 P 6500 2100
-F 0 "J?" H 6392 1375 50  0000 C CNN
+F 0 "J5" H 6392 1375 50  0000 C CNN
 F 1 "SERIAL_HEADER" H 6392 1466 50  0000 C CNN
 F 2 "Connector_PinHeader_1.27mm:PinHeader_1x10_P1.27mm_Vertical" H 6500 2100 50  0001 C CNN
@@
 	5500 1700 6300 1700
 $Comp
-L power:+5V #PWR?
+L power:+5V #PWR0123
 U 1 1 5D0A14B8
 P 2850 1450
-F 0 "#PWR?" H 2850 1300 50  0001 C CNN
+F 0 "#PWR0123" H 2850 1300 50  0001 C CNN
 F 1 "+5V" H 2865 1623 50  0000 C CNN
 F 2 "" H 2850 1450 50  0001 C CNN
@@
 Connection ~ 2850 1600
 $Comp
-L power:+5V #PWR?
+L power:+5V #PWR0124
 U 1 1 5D0A9573
 P 4550 1050
-F 0 "#PWR?" H 4550 900 50  0001 C CNN
+F 0 "#PWR0124" H 4550 900 50  0001 C CNN
 F 1 "+5V" V 4565 1178 50  0000 L CNN
 F 2 "" H 4550 1050 50  0001 C CNN
@@
 $EndComp
 $Comp
-L power:GND #PWR?
+L power:GND #PWR0125
 U 1 1 5D0A9D8F
 P 5150 1050
-F 0 "#PWR?" H 5150 800 50  0001 C CNN
+F 0 "#PWR0125" H 5150 800 50  0001 C CNN
 F 1 "GND" V 5155 922 50  0000 R CNN
 F 2 "" H 5150 1050 50  0001 C CNN
@@
 $EndComp
 $Comp
-L taobao-c:C475,0603 C?
+L taobao-c:C475,0603 C4
 U 1 1 5D0AA385
 P 4850 1050
-F 0 "C?" V 4621 1050 50  0000 C CNN
+F 0 "C4" V 4621 1050 50  0000 C CNN
 F 1 "C475,0603" V 4712 1050 50  0000 C CNN
 F 2 "Capacitor_SMD:C_0603_1608Metric_Pad1.05x0.95mm_HandSolder" H 4850 1050 50  0001 C CNN
@@
 	6300 2400 6050 2400
 $Comp
-L power:+5V #PWR?
+L power:+5V #PWR0126
 U 1 1 5D0A562E
 P 6050 2750
-F 0 "#PWR?" H 6050 2600 50  0001 C CNN
+F 0 "#PWR0126" H 6050 2600 50  0001 C CNN
 F 1 "+5V" H 6065 2923 50  0000 C CNN
 F 2 "" H 6050 2750 50  0001 C CNN
@@
 	6200 2700 6200 2500
 $Comp
-L power:GND #PWR?
+L power:GND #PWR0127
 U 1 1 5D09B4B9
 P 6200 2700
-F 0 "#PWR?" H 6200 2450 50  0001 C CNN
+F 0 "#PWR0127" H 6200 2450 50  0001 C CNN
 F 1 "GND" H 6205 2527 50  0000 C CNN
 F 2 "" H 6200 2700 50  0001 C CNN
@@
 $EndBitmap
 $Comp
-L power:GND #PWR?
+L power:GND #PWR0128
 U 1 1 5D0516E0
 P 1550 2750
-F 0 "#PWR?" H 1550 2500 50  0001 C CNN
+F 0 "#PWR0128" H 1550 2500 50  0001 C CNN
 F 1 "GND" H 1555 2577 50  0000 C CNN
 F 2 "" H 1550 2750 50  0001 C CNN
@@
 	1550 2500 1550 2750
 $Comp
-L power:GND #PWR?
+L power:GND #PWR0129
 U 1 1 5D057019
 P 2650 2750
-F 0 "#PWR?" H 2650 2500 50  0001 C CNN
+F 0 "#PWR0129" H 2650 2500 50  0001 C CNN
 F 1 "GND" H 2655 2577 50  0000 C CNN
 F 2 "" H 2650 2750 50  0001 C CNN
@@
 $EndBitmap
 $Comp
-L my_solder_jumper:SolderJumper_2_Open_round JP?
+L my_solder_jumper:SolderJumper_2_Open_round JP4
 U 1 1 5D10712E
 P 5700 2850
-F 0 "JP?" V 5750 2550 50  0000 L CNN
+F 0 "JP4" V 5750 2550 50  0000 L CNN
 F 1 "SLEEP_EN" V 5850 2300 50  0000 L CNN
 F 2 "Jumper:SolderJumper-2_P1.3mm_Open_RoundedPad1.0x1.5mm" H 5700 2850 50  0001 C CNN
@@
 $EndComp
 $Comp
-L power:GND #PWR?
+L power:GND #PWR0130
 U 1 1 5D107B8C
 P 5700 3150
-F 0 "#PWR?" H 5700 2900 50  0001 C CNN
+F 0 "#PWR0130" H 5700 2900 50  0001 C CNN
 F 1 "GND" H 5750 2950 50  0000 C CNN
 F 2 "" H 5700 3150 50  0001 C CNN
