File: hardware/ESP12_button.sch (KiCad schematic (older format))
At the start: 7 parts

Commit message: update,
Parts:
- gave numbers to parts that had none: 7
Changed lines of the file:
@@
 AR Path="/5CD03534/5CD6BE5F/5CD6EFDD" Ref="#PWR?"  Part="1"
 AR Path="/5CD47361/5CD6BE5F/5CD6EFDD" Ref="#PWR?"  Part="1"
-AR Path="/5CF23C1A/5CD6BE5F/5CD6EFDD" Ref="#PWR?"  Part="1"
-F 0 "#PWR?" H 3350 950 50  0001 C CNN
+AR Path="/5CF23C1A/5CD6BE5F/5CD6EFDD" Ref="#PWR0134"  Part="1"
+F 0 "#PWR0134" H 3350 950 50  0001 C CNN
 F 1 "+3V3" H 3400 1300 50  0000 C CNN
 F 2 "" H 3350 1100 50  0001 C CNN
@@
 AR Path="/5CD03534/5CD6BE5F/5CD6F2CA" Ref="R?"  Part="1"
 AR Path="/5CD47361/5CD6BE5F/5CD6F2CA" Ref="R?"  Part="1"
-AR Path="/5CF23C1A/5CD6BE5F/5CD6F2CA" Ref="R?"  Part="1"
-F 0 "R?" H 3450 1450 50  0000 L CNN
+AR Path="/5CF23C1A/5CD6BE5F/5CD6F2CA" Ref="R12"  Part="1"
+F 0 "R12" H 3450 1450 50  0000 L CNN
 F 1 "R471,0603" H 3450 1400 50  0000 L CNN
 F 2 "Resistor_SMD:R_0603_1608Metric_Pad1.05x0.95mm_HandSolder" H 3350 1400 50  0001 C CNN
@@
 AR Path="/5CD03534/5CD6BE5F/5CD6F699" Ref="D?"  Part="1"
 AR Path="/5CD47361/5CD6BE5F/5CD6F699" Ref="D?"  Part="1"
-AR Path="/5CF23C1A/5CD6BE5F/5CD6F699" Ref="D?"  Part="1"
-F 0 "D?" V 3400 1650 50  0000 R CNN
+AR Path="/5CF23C1A/5CD6BE5F/5CD6F699" Ref="D2"  Part="1"
+F 0 "D2" V 3400 1650 50  0000 R CNN
 F 1 "LED_BLUE,0603" V 3350 1650 50  0000 R CNN
 F 2 "LED_SMD:LED_0603_1608Metric_Pad1.05x0.95mm_HandSolder" V 3350 1750 50  0001 C CNN
@@
 AR Path="/5CD03534/5CD6BE5F/5CD70197" Ref="R?"  Part="1"
 AR Path="/5CD47361/5CD6BE5F/5CD70197" Ref="R?"  Part="1"
-AR Path="/5CF23C1A/5CD6BE5F/5CD70197" Ref="R?"  Part="1"
-F 0 "R?" H 3450 2200 50  0000 L CNN
+AR Path="/5CF23C1A/5CD6BE5F/5CD70197" Ref="R14"  Part="1"
+F 0 "R14" H 3450 2200 50  0000 L CNN
 F 1 "R0,0603" H 3450 2150 50  0000 L CNN
 F 2 "Resistor_SMD:R_0603_1608Metric_Pad1.05x0.95mm_HandSolder" H 3350 2150 50  0001 C CNN
@@
 AR Path="/5CD03534/5CD6BE5F/5CD705A6" Ref="SW?"  Part="1"
 AR Path="/5CD47361/5CD6BE5F/5CD705A6" Ref="SW?"  Part="1"
-AR Path="/5CF23C1A/5CD6BE5F/5CD705A6" Ref="SW?"  Part="1"
-F 0 "SW?" V 3600 2800 50  0000 L CNN
+AR Path="/5CF23C1A/5CD6BE5F/5CD705A6" Ref="SW5"  Part="1"
+F 0 "SW5" V 3600 2800 50  0000 L CNN
 F 1 "RST" V 3650 2800 50  0000 L CNN
 F 2 "footprint-lib:SW_SPST_CK_RS282G05A3" H 3650 2850 50  0001 C CNN
@@
 AR Path="/5CD03534/5CD6BE5F/5CD70C90" Ref="R?"  Part="1"
 AR Path="/5CD47361/5CD6BE5F/5CD70C90" Ref="R?"  Part="1"
-AR Path="/5CF23C1A/5CD6BE5F/5CD70C90" Ref="R?"  Part="1"
-F 0 "R?" H 4000 2200 50  0000 L CNN
+AR Path="/5CF23C1A/5CD6BE5F/5CD70C90" Ref="R15"  Part="1"
+F 0 "R15" H 4000 2200 50  0000 L CNN
 F 1 "R471,0603" H 4000 2150 50  0000 L CNN
 F 2 "Resistor_SMD:R_0603_1608Metric_Pad1.05x0.95mm_HandSolder" H 3900 2150 50  0001 C CNN
@@
 AR Path="/5CD03534/5CD6BE5F/5CD72E50" Ref="#PWR?"  Part="1"
 AR Path="/5CD47361/5CD6BE5F/5CD72E50" Ref="#PWR?"  Part="1"
-AR Path="/5CF23C1A/5CD6BE5F/5CD72E50" Ref="#PWR?"  Part="1"
-F 0 "#PWR?" H 3650 2800 50  0001 C CNN
+AR Path="/5CF23C1A/5CD6BE5F/5CD72E50" Ref="#PWR0153"  Part="1"
+F 0 "#PWR0153" H 3650 2800 50  0001 C CNN
 F 1 "GND" H 3700 2850 50  0000 C CNN
 F 2 "" H 3650 3050 50  0001 C CNN
@@
 AR Path="/5CD03534/5CD6BE5F/5CD73ECF" Ref="SW?"  Part="1"
 AR Path="/5CD47361/5CD6BE5F/5CD73ECF" Ref="SW?"  Part="1"
-AR Path="/5CF23C1A/5CD6BE5F/5CD73ECF" Ref="SW?"  Part="1"
-F 0 "SW?" V 5000 2550 50  0000 L CNN
+AR Path="/5CF23C1A/5CD6BE5F/5CD73ECF" Ref="SW4"  Part="1"
+F 0 "SW4" V 5000 2550 50  0000 L CNN
 F 1 "FLASH" V 5050 2550 50  0000 L CNN
 F 2 "footprint-lib:SW_SPST_CK_RS282G05A3" H 5050 2600 50  0001 C CNN
@@
 AR Path="/5CD03534/5CD6BE5F/5CD75A97" Ref="#PWR?"  Part="1"
 AR Path="/5CD47361/5CD6BE5F/5CD75A97" Ref="#PWR?"  Part="1"
-AR Path="/5CF23C1A/5CD6BE5F/5CD75A97" Ref="#PWR?"  Part="1"
-F 0 "#PWR?" H 5050 2550 50  0001 C CNN
+AR Path="/5CF23C1A/5CD6BE5F/5CD75A97" Ref="#PWR0154"  Part="1"
+F 0 "#PWR0154" H 5050 2550 50  0001 C CNN
 F 1 "GND" H 5100 2600 50  0000 C CNN
 F 2 "" H 5050 2800 50  0001 C CNN
@@
 AR Path="/5CD03534/5CD6BE5F/5CD7498A" Ref="R?"  Part="1"
 AR Path="/5CD47361/5CD6BE5F/5CD7498A" Ref="R?"  Part="1"
-AR Path="/5CF23C1A/5CD6BE5F/5CD7498A" Ref="R?"  Part="1"
-F 0 "R?" H 5150 2000 50  0000 L CNN
+AR Path="/5CF23C1A/5CD6BE5F/5CD7498A" Ref="R13"  Part="1"
+F 0 "R13" H 5150 2000 50  0000 L CNN
 F 1 "R471,0603" H 5150 1950 50  0000 L CNN
 F 2 "Resistor_SMD:R_0603_1608Metric_Pad1.05x0.95mm_HandSolder" H 5050 1950 50  0001 C CNN
