File: hardware/SHT3X.sch (KiCad schematic (older format))
At the start: 6 parts, among them J1 SHT3x_HEADER, U1 SHT3x-DIS

Commit message: update,
Parts:
- JP?: renamed from JP1; value SolderJumper_2_Open_round -> SCL_SDA
- renumbered C1 to C?, J1 to J?, JP2 to JP?, RN1 to RN?, U1 to U?
Connections:
- net ALERT: now also J?.6 (Pin_6); no longer J?.5 (Pin_5)
- net NRST: now also J?.3 (Pin_3), RN?.4 (R4.1); no longer J?.6 (Pin_6), RN?.2 (R2.1)
- net SCL: now also J?.5 (Pin_5); no longer J?.4 (Pin_4)
- net SDA: now also J?.4 (Pin_4), RN?.2 (R2.1); no longer J?.3 (Pin_3), RN?.4 (R4.1)

Commit message: update,
Parts:
- gave numbers to parts that had none: 6
Changed lines of the file:
@@
 $EndBitmap
 $Comp
-L taobao-components:SHT3x-DIS U?
+L taobao-components:SHT3x-DIS U1
 U 1 1 5CFA0226
 P 3750 2150
-F 0 "U?" H 3750 2715 50  0000 C CNN
+F 0 "U1" H 3750 2715 50  0000 C CNN
 F 1 "SHT3x-DIS" H 3750 2624 50  0000 C CNN
 F 2 "footprint-lib:SHT3x-DIS" H 4550 1500 50  0001 C CNN
@@
 $EndComp
 $Comp
-L power:GND #PWR?
+L power:GND #PWR0101
 U 1 1 5CFA0C01
 P 3750 3050
-F 0 "#PWR?" H 3750 2800 50  0001 C CNN
+F 0 "#PWR0101" H 3750 2800 50  0001 C CNN
 F 1 "GND" H 3755 2877 50  0000 C CNN
 F 2 "" H 3750 3050 50  0001 C CNN
@@
 $EndComp
 $Comp
-L power:GND #PWR?
+L power:GND #PWR0102
 U 1 1 5CFA0FDE
 P 2950 3050
-F 0 "#PWR?" H 2950 2800 50  0001 C CNN
+F 0 "#PWR0102" H 2950 2800 50  0001 C CNN
 F 1 "GND" H 2955 2877 50  0000 C CNN
 F 2 "" H 2950 3050 50  0001 C CNN
@@
 $EndComp
 $Comp
-L power:GND #PWR?
+L power:GND #PWR0103
 U 1 1 5CFA11DA
 P 4600 3050
-F 0 "#PWR?" H 4600 2800 50  0001 C CNN
+F 0 "#PWR0103" H 4600 2800 50  0001 C CNN
 F 1 "GND" H 4605 2877 50  0000 C CNN
 F 2 "" H 4600 3050 50  0001 C CNN
@@
 	2950 2450 3100 2450
 $Comp
-L taobao-rpack:RN_472,0603 RN?
+L taobao-rpack:RN_472,0603 RN1
 U 1 1 5CFA1908
 P 2050 1500
-F 0 "RN?" H 2238 1546 50  0000 L CNN
+F 0 "RN1" H 2238 1546 50  0000 L CNN
 F 1 "RN_472,0603" H 2238 1455 50  0000 L CNN
 F 2 "Resistor_SMD:R_Array_Concave_4x0603" V 2325 1500 50  0001 C CNN
@@
 	4400 2250 4900 2250
 $Comp
-L power:+3V3 #PWR?
+L power:+3V3 #PWR0104
 U 1 1 5CFA3064
 P 1900 650
-F 0 "#PWR?" H 1900 500 50  0001 C CNN
+F 0 "#PWR0104" H 1900 500 50  0001 C CNN
 F 1 "+3V3" H 1915 823 50  0000 C CNN
 F 2 "" H 1900 650 50  0001 C CNN
@@
 $EndComp
 $Comp
-L my_solder_jumper:SolderJumper_2_Open_round JP?
+L my_solder_jumper:SolderJumper_2_Open_round JP1
 U 1 1 5CFA372A
 P 1900 1000
-F 0 "JP?" V 1850 900 50  0000 R CNN
+F 0 "JP1" V 1850 900 50  0000 R CNN
 F 1 "SCL_SDA" V 1900 900 50  0000 R CNN
 F 2 "Jumper:SolderJumper-2_P1.3mm_Open_RoundedPad1.0x1.5mm" H 1900 1000 50  0001 C CNN
@@
 Connection ~ 1900 1200
 $Comp
-L power:+3V3 #PWR?
+L power:+3V3 #PWR0105
 U 1 1 5CFA5513
 P 4600 1600
-F 0 "#PWR?" H 4600 1450 50  0001 C CNN
+F 0 "#PWR0105" H 4600 1450 50  0001 C CNN
 F 1 "+3V3" H 4615 1773 50  0000 C CNN
 F 2 "" H 4600 1600 50  0001 C CNN
@@
 	4600 1850 4600 1600
 $Comp
-L power:+3V3 #PWR?
+L power:+3V3 #PWR0106
 U 1 1 5CFA6101
 P 3450 1350
-F 0 "#PWR?" H 3450 1200 50  0001 C CNN
+F 0 "#PWR0106" H 3450 1200 50  0001 C CNN
 F 1 "+3V3" V 3465 1478 50  0000 L CNN
 F 2 "" H 3450 1350 50  0001 C CNN
@@
 $EndComp
 $Comp
-L power:GND #PWR?
+L power:GND #PWR0107
 U 1 1 5CFA6490
 P 4000 1350
-F 0 "#PWR?" H 4000 1100 50  0001 C CNN
+F 0 "#PWR0107" H 4000 1100 50  0001 C CNN
 F 1 "GND" V 4005 1222 50  0000 R CNN
 F 2 "" H 4000 1350 50  0001 C CNN
@@
 $EndComp
 $Comp
-L taobao-c:C104,0805 C?
+L taobao-c:C104,0805 C1
 U 1 1 5CFA71B1
 P 3700 1350
-F 0 "C?" V 3471 1350 50  0000 C CNN
+F 0 "C1" V 3471 1350 50  0000 C CNN
 F 1 "C104,0805" V 3562 1350 50  0000 C CNN
 F 2 "Capacitor_SMD:C_0805_2012Metric_Pad1.15x1.40mm_HandSolder" H 3700 1350 50  0001 C CNN
@@
 ADDR
 $Comp
-L my_solder_jumper:SolderJumper_2_Open_round JP?
+L my_solder_jumper:SolderJumper_2_Open_round JP2
 U 1 1 5CFABF79
 P 2300 2550
-F 0 "JP?" V 2254 2618 50  0000 L CNN
+F 0 "JP2" V 2254 2618 50  0000 L CNN
 F 1 "J_ADDR" V 2345 2618 50  0000 L CNN
 F 2 "Jumper:SolderJumper-2_P1.3mm_Open_RoundedPad1.0x1.5mm" H 2300 2550 50  0001 C CNN
@@
 $EndComp
 $Comp
-L power:GND #PWR?
+L power:GND #PWR0108
 U 1 1 5CFAC548
 P 2300 3050
-F 0 "#PWR?" H 2300 2800 50  0001 C CNN
+F 0 "#PWR0108" H 2300 2800 50  0001 C CNN
 F 1 "GND" H 2305 2877 50  0000 C CNN
 F 2 "" H 2300 3050 50  0001 C CNN
@@
 	1950 1700 1950 2050
 $Comp
-L Connector:Conn_01x06_Female J?
+L Connector:Conn_01x06_Female J1
 U 1 1 5CFBB0DE
 P 1250 2750
-F 0 "J?" H 1142 3135 50  0000 C CNN
+F 0 "J1" H 1142 3135 50  0000 C CNN
 F 1 "SHT3x_HEADER" H 1142 3044 50  0000 C CNN
 F 2 "Connector_PinHeader_1.27mm:PinHeader_1x06_P1.27mm_Vertical" H 1250 2750 50  0001 C CNN
@@
 $EndComp
 $Comp
-L power:GND #PWR?
+L power:GND #PWR0109
 U 1 1 5CFBC187
 P 1600 2400
-F 0 "#PWR?" H 1600 2150 50  0001 C CNN
+F 0 "#PWR0109" H 1600 2150 50  0001 C CNN
 F 1 "GND" H 1605 2227 50  0000 C CNN
 F 2 "" H 1600 2400 50  0001 C CNN
@@
 	1600 2550 1450 2550
 $Comp
-L power:+3V3 #PWR?
+L power:+3V3 #PWR0110
 U 1 1 5CFBE976
 P 1800 2350
-F 0 "#PWR?" H 1800 2200 50  0001 C CNN
+F 0 "#PWR0110" H 1800 2200 50  0001 C CNN
 F 1 "+3V3" H 1815 2523 50  0000 C CNN
 F 2 "" H 1800 2350 50  0001 C CNN
