File: hardware/esp12_core.sch (KiCad schematic (older format))
At the start: 16 parts, among them J2 I2C_HEADER,2.54, J3 I2C_HEADER, U2 ESP12

Commit message: update,
Parts:
- added Q? (x2): SS9013_J3, footprint-lib:9013,J3,SOT23, symbol taobao-transistor:SS9013_J3
- added R? (x2): R123,0603, Resistor_SMD:R_0603_1608Metric_Pad1.05x0.95mm_HandSolder, symbol taobao-r:R123,0603
Connections:
- net nRST: now also Q?.3 (C)
- net GPIO0 renamed FAN_PWM
- net FAN_PWM: now also Q?.3 (C)
- new net: Q?.1 (B), R?.2 (x2)
- new net DTR: Q?.2 (E), R?.1
- new net RTS: Q?.2 (E), R?.1
- no-connect marks 9 -> 13
Other:
- note added: "5V TO 3V3 LEVEL SWITCH"
- moved on the sheet: J3, RN2, TP1, TP2

Commit message: update,
Parts:
- gave numbers to parts that had none: 4
Changed lines of the file:
@@
 AR Path="/5CD47361/5CD5414F/5D120566" Ref="Q?"  Part="1"
 AR Path="/5CF23C1A/5CD5414F/5D120566" Ref="Q?"  Part="1"
-AR Path="/5CF23C1A/5D120566" Ref="Q?"  Part="1"
-F 0 "Q?" H 8300 4700 50  0000 L CNN
+AR Path="/5CF23C1A/5D120566" Ref="Q1"  Part="1"
+F 0 "Q1" H 8300 4700 50  0000 L CNN
 F 1 "SS9013_J3" H 8300 4650 50  0000 L CNN
 F 2 "footprint-lib:9013,J3,SOT23" H 8300 4575 50  0001 L CIN
@@
 AR Path="/5CD47361/5CD5414F/5D12056C" Ref="Q?"  Part="1"
 AR Path="/5CF23C1A/5CD5414F/5D12056C" Ref="Q?"  Part="1"
-AR Path="/5CF23C1A/5D12056C" Ref="Q?"  Part="1"
-F 0 "Q?" H 8300 5350 50  0000 L CNN
+AR Path="/5CF23C1A/5D12056C" Ref="Q2"  Part="1"
+F 0 "Q2" H 8300 5350 50  0000 L CNN
 F 1 "SS9013_J3" H 8300 5400 50  0000 L CNN
 F 2 "footprint-lib:9013,J3,SOT23" H 8300 5325 50  0001 L CIN
@@
 AR Path="/5CD47361/5CD5414F/5D12057E" Ref="R?"  Part="1"
 AR Path="/5CF23C1A/5CD5414F/5D12057E" Ref="R?"  Part="1"
-AR Path="/5CF23C1A/5D12057E" Ref="R?"  Part="1"
-F 0 "R?" V 8300 4650 50  0000 C CNN
+AR Path="/5CF23C1A/5D12057E" Ref="R7"  Part="1"
+F 0 "R7" V 8300 4650 50  0000 C CNN
 F 1 "R123,0603" V 8400 4650 50  0000 C CNN
 F 2 "Resistor_SMD:R_0603_1608Metric_Pad1.05x0.95mm_HandSolder" H 8550 4650 50  0001 C CNN
@@
 AR Path="/5CD47361/5CD5414F/5D120584" Ref="R?"  Part="1"
 AR Path="/5CF23C1A/5CD5414F/5D120584" Ref="R?"  Part="1"
-AR Path="/5CF23C1A/5D120584" Ref="R?"  Part="1"
-F 0 "R?" V 8300 5400 50  0000 C CNN
+AR Path="/5CF23C1A/5D120584" Ref="R8"  Part="1"
+F 0 "R8" V 8300 5400 50  0000 C CNN
 F 1 "R123,0603" V 8400 5400 50  0000 C CNN
 F 2 "Resistor_SMD:R_0603_1608Metric_Pad1.05x0.95mm_HandSolder" H 8550 5400 50  0001 C CNN
