File: hardware/motor.sch (KiCad schematic (older format))
At the start: 0 parts

Commit message: update,
Parts:
- added C?: C106,0805, Capacitor_SMD:C_0805_2012Metric_Pad1.15x1.40mm_HandSolder, symbol taobao-c:C106,0805
- added D?: EN, LED_SMD:LED_0603_1608Metric_Pad1.05x0.95mm_HandSolder, symbol taobao-led:LED_BLUE,0603
- added J?: FAN0, footprint-lib:XH_TEMPERATURE_SENSOR_TERMINAL_2.54, symbol Connector:Screw_Terminal_01x02
- added Q?: D882, footprint-lib:SOT-89-3,thermal_vias, symbol taobao-components:D882
- added R?: R104,0805, Resistor_SMD:R_0805_2012Metric_Pad1.15x1.40mm_HandSolder, symbol taobao-r:R104,0805
- added R?: R182,0603, Resistor_SMD:R_0603_1608Metric_Pad1.05x0.95mm_HandSolder, symbol taobao-r:R182,0603
- added R?: R100,0805, Resistor_SMD:R_0805_2012Metric_Pad1.15x1.40mm_HandSolder, symbol taobao-r:R100,0805
- added R?: R100,0603, Resistor_SMD:R_0603_1608Metric_Pad1.05x0.95mm_HandSolder, symbol taobao-r:R100,0603
- added TP?: FAN0_EN_TP, Connector_PinHeader_1.00mm:PinHeader_1x01_P1.00mm_Vertical, symbol Connector:TestPoint
Connections:
- new net: Q?.1 (B), R?.1
- new net: Q?.2 (C), R?.2
- new net: D?.2 (A), R?.1
- new net +12V: C?.1, J?.1 (Pin_1), R?.2
- new net FAN0_EN: R?.2, R?.2, TP?.1
- new net FAN0_N: C?.2, D?.1 (K), J?.2 (Pin_2), R?.1
- new net GND: Q?.3 (E), R?.1
Other:
- note added: "optional"

Commit message: update,
Parts:
- gave numbers to parts that had none: 9
Changed lines of the file:
@@
 AR Path="/5CC242F9" Ref="J?"  Part="1"
 AR Path="/5CC2401E/5CE37797/5CC242F9" Ref="J?"  Part="1"
-AR Path="/5D0F9966/5CC242F9" Ref="J?"  Part="1"
-F 0 "J?" H 6950 1250 50  0000 C CNN
+AR Path="/5D0F9966/5CC242F9" Ref="J6"  Part="1"
+F 0 "J6" H 6950 1250 50  0000 C CNN
 F 1 "FAN0" H 6950 1350 50  0000 C CNN
 F 2 "footprint-lib:XH_TEMPERATURE_SENSOR_TERMINAL_2.54" H 7000 1600 50  0001 C CNN
@@
 AR Path="/5CC8A042" Ref="R?"  Part="1"
 AR Path="/5CC2401E/5CE37797/5CC8A042" Ref="R?"  Part="1"
-AR Path="/5D0F9966/5CC8A042" Ref="R?"  Part="1"
-F 0 "R?" V 4354 2350 50  0000 C CNN
+AR Path="/5D0F9966/5CC8A042" Ref="R23"  Part="1"
+F 0 "R23" V 4354 2350 50  0000 C CNN
 F 1 "R100,0805" V 4445 2350 50  0000 C CNN
 F 2 "Resistor_SMD:R_0805_2012Metric_Pad1.15x1.40mm_HandSolder" H 4550 2350 50  0001 C CNN
@@
 AR Path="/5CC8A033" Ref="R?"  Part="1"
 AR Path="/5CC2401E/5CE37797/5CC8A033" Ref="R?"  Part="1"
-AR Path="/5D0F9966/5CC8A033" Ref="R?"  Part="1"
-F 0 "R?" V 4354 2750 50  0000 C CNN
+AR Path="/5D0F9966/5CC8A033" Ref="R24"  Part="1"
+F 0 "R24" V 4354 2750 50  0000 C CNN
 F 1 "R104,0805" V 4445 2750 50  0000 C CNN
 F 2 "Resistor_SMD:R_0805_2012Metric_Pad1.15x1.40mm_HandSolder" H 4550 2750 50  0001 C CNN
@@
 AR Path="/5CC242FE" Ref="#PWR?"  Part="1"
 AR Path="/5CC2401E/5CE37797/5CC242FE" Ref="#PWR?"  Part="1"
-AR Path="/5D0F9966/5CC242FE" Ref="#PWR?"  Part="1"
-F 0 "#PWR?" H 5300 2700 50  0001 C CNN
+AR Path="/5D0F9966/5CC242FE" Ref="#PWR0166"  Part="1"
+F 0 "#PWR0166" H 5300 2700 50  0001 C CNN
 F 1 "GND" H 5305 2777 50  0000 C CNN
 F 2 "" H 5300 2950 50  0001 C CNN
@@
 AR Path="/5CC8A037" Ref="R?"  Part="1"
 AR Path="/5CC2401E/5CE37797/5CC8A037" Ref="R?"  Part="1"
-AR Path="/5D0F9966/5CC8A037" Ref="R?"  Part="1"
-F 0 "R?" H 5859 1246 50  0000 L CNN
+AR Path="/5D0F9966/5CC8A037" Ref="R21"  Part="1"
+F 0 "R21" H 5859 1246 50  0000 L CNN
 F 1 "R182,0603" H 5859 1155 50  0000 L CNN
 F 2 "Resistor_SMD:R_0603_1608Metric_Pad1.05x0.95mm_HandSolder" H 5800 1200 50  0001 C CNN
@@
 AR Path="/5CC242FF" Ref="#PWR?"  Part="1"
 AR Path="/5CC2401E/5CE37797/5CC242FF" Ref="#PWR?"  Part="1"
-AR Path="/5D0F9966/5CC242FF" Ref="#PWR?"  Part="1"
-F 0 "#PWR?" H 6050 750 50  0001 C CNN
+AR Path="/5D0F9966/5CC242FF" Ref="#PWR0167"  Part="1"
+F 0 "#PWR0167" H 6050 750 50  0001 C CNN
 F 1 "+12V" H 6065 1073 50  0000 C CNN
 F 2 "" H 6050 900 50  0001 C CNN
@@
 AR Path="/5CC8A044" Ref="D?"  Part="1"
 AR Path="/5CC2401E/5CE37797/5CC8A044" Ref="D?"  Part="1"
-AR Path="/5D0F9966/5CC8A044" Ref="D?"  Part="1"
-F 0 "D?" V 5754 1598 50  0000 L CNN
+AR Path="/5D0F9966/5CC8A044" Ref="D9"  Part="1"
+F 0 "D9" V 5754 1598 50  0000 L CNN
 F 1 "EN" V 5845 1598 50  0000 L CNN
 F 2 "LED_SMD:LED_0603_1608Metric_Pad1.05x0.95mm_HandSolder" V 5800 1500 50  0001 C CNN
@@
 AR Path="/5CC2401E/5CC242A1/5CC87678" Ref="Q?"  Part="1"
 AR Path="/5CC2401E/5CE37797/5CC87678" Ref="Q?"  Part="1"
-AR Path="/5D0F9966/5CC87678" Ref="Q?"  Part="1"
-F 0 "Q?" H 5400 2400 50  0000 L CNN
+AR Path="/5D0F9966/5CC87678" Ref="Q3"  Part="1"
+F 0 "Q3" H 5400 2400 50  0000 L CNN
 F 1 "D882" H 5400 2350 50  0000 L CNN
 F 2 "footprint-lib:SOT-89-3,thermal_vias" H 5400 2450 50  0001 C CNN
@@
 AR Path="/5CC2401E/5CC242A1/5CC8A048" Ref="R?"  Part="1"
 AR Path="/5CC2401E/5CE37797/5CC8A048" Ref="R?"  Part="1"
-AR Path="/5D0F9966/5CC8A048" Ref="R?"  Part="1"
-F 0 "R?" H 5400 2000 50  0000 L CNN
+AR Path="/5D0F9966/5CC8A048" Ref="R22"  Part="1"
+F 0 "R22" H 5400 2000 50  0000 L CNN
 F 1 "R100,0603" H 5400 1950 50  0000 L CNN
 F 2 "Resistor_SMD:R_0603_1608Metric_Pad1.05x0.95mm_HandSolder" H 5300 1950 50  0001 C CNN
@@
 FAN0_N
 $Comp
-L Connector:TestPoint TP?
+L Connector:TestPoint TP5
 U 1 1 5CE017DB
 P 3850 2200
-F 0 "TP?" H 3950 2350 50  0000 L CNN
+F 0 "TP5" H 3950 2350 50  0000 L CNN
 F 1 "FAN0_EN_TP" H 3950 2250 50  0000 L CNN
 F 2 "Connector_PinHeader_1.00mm:PinHeader_1x01_P1.00mm_Vertical" H 4050 2200 50  0001 C CNN
@@
 optional
 $Comp
-L taobao-c:C106,0805 C?
+L taobao-c:C106,0805 C16
 U 1 1 5D0A9ED8
 P 5450 1300
-F 0 "C?" H 5542 1346 50  0000 L CNN
+F 0 "C16" H 5542 1346 50  0000 L CNN
 F 1 "C106,0805" H 5542 1255 50  0000 L CNN
 F 2 "Capacitor_SMD:C_0805_2012Metric_Pad1.15x1.40mm_HandSolder" H 5450 1300 50  0001 C CNN
